Commit message: update urdf

File: robotic_arm_v4_urdf/urdf/robotic_arm_v4_urdf.urdf (robot description, URDF)
Before this commit: robot robotic_arm_v4_urdf, 7 links, 6 joints
Joints:
- joint Joint1: origin xyz=0 0 0 rpy=1.5707963267949 0 0.127561037294902 -> xyz=0 0 0 rpy=1.5707963267949 0 0
- joint Joint2: origin xyz=0 0.0729999999999994 0 rpy=0 0 -0.716850557781711 -> xyz=0 0.0729999999999994 0 rpy=0 0 -0.705
- joint Joint3: origin xyz=-0.20761 0.24351 0 rpy=0.85395 -1.5708 0 -> xyz=-0.20761 0.24351 0 rpy=-0.86 -1.5708 0

Commit message: update urdf

File: robotic_arm_v4_urdf/urdf/robotic_arm_v4_urdf.urdf (robot description, URDF)
Before this commit: robot robotic_arm_v4_urdf, 7 links, 6 joints
Links:
- link End_Effector: geometry collision box size=0.06 0.06 0.06; visual mesh filename=package://robotic_arm_v4_urdf/meshes/End_Effector.STL
- link J3_J4: geometry collision box size=0.10 0.16 0.10; visual mesh filename=package://robotic_arm_v4_urdf/meshes/J3_J4.STL
- link J5_J6: geometry collision box size=0.08 0.04 0.08; visual mesh filename=package://robotic_arm_v4_urdf/meshes/J5_J6.STL
- link Link0: geometry collision box size=0.12 0.12 0.12; visual mesh filename=package://robotic_arm_v4_urdf/meshes/Link0.STL
- link Link1: geometry collision box size=0.24 0.28 0.08; visual mesh filename=package://robotic_arm_v4_urdf/meshes/Link1.STL
- link Link2: geometry collision box size=0.08 0.26 0.08; visual mesh filename=package://robotic_arm_v4_urdf/meshes/Link2.STL
- link base_link: geometry collision box size=0.15 0.05 0.15; visual mesh filename=package://robotic_arm_v4_urdf/meshes/base_link.STL

Commit message: update collision mesh

File: robotic_arm_v4_urdf/urdf/robotic_arm_v4_urdf.urdf (robot description, URDF)
Before this commit: robot robotic_arm_v4_urdf, 7 links, 6 joints
Links:
- link End_Effector: geometry collision box size=0.15 0.14 0.06; visual mesh filename=package://robotic_arm_v4_urdf/meshes/End_Effector.STL
- link J3_J4: geometry collision box size=0.065 0.20 0.16; visual mesh filename=package://robotic_arm_v4_urdf/meshes/J3_J4.STL
- link J5_J6: geometry collision cylinder length=0.14 radius=0.04; visual mesh filename=package://robotic_arm_v4_urdf/meshes/J5_J6.STL
- link Link0: geometry collision box size=0.12 0.12 0.07; visual mesh filename=package://robotic_arm_v4_urdf/meshes/Link0.STL
- link Link1: geometry collision box size=0.08 0.40 0.035; visual mesh filename=package://robotic_arm_v4_urdf/meshes/Link1.STL
- link Link2: geometry collision box size=0.12 0.20 0.08; visual mesh filename=package://robotic_arm_v4_urdf/meshes/Link2.STL
- link base_link: geometry collision box size=0.2 0.10 0.07; visual mesh filename=package://robotic_arm_v4_urdf/meshes/base_link.STL

Commit message: feat(control): add collision-aware homing and enforce joint limits
choose homing groups dynamically from Joint2 angle to reduce collision
risk during homing
remove static homing_order / homing_groups config usage and log selected
runtime sequence
update README homing section to document the new angle-based sequence
switch URDF joints from continuous to revolute and define per-joint
position/velocity limits
enable matching position limits in joint_limits.yaml for all 6 joints
improve mcu_emulator.py startup behavior: raw PTY mode, startup grace
period, and first-frame timing log
add AGENTS.md and CLAUDE.md GitNexus guidance, and ignore .claude in
.gitignore

File: robotic_arm_v4_urdf/urdf/robotic_arm_v4_urdf.urdf (robot description, URDF)
Before this commit: robot robotic_arm_v4_urdf, 7 links, 6 joints
Joints:
- joint Joint1: limit lower=-3.14 upper=3.14 effort=6 velocity=60 -> lower=-3.14159 upper=3.14159 effort=6 velocity=1.2; type continuous -> revolute
- joint Joint2: limit lower=-3.14 upper=3.14 effort=40 velocity=70 -> lower=-1.5708 upper=1.5708 effort=40 velocity=1.2; type continuous -> revolute
- joint Joint3: limit lower=-3.14 upper=3.14 effort=40 velocity=70 -> lower=-1.20 upper=4.0 effort=40 velocity=1.2; type continuous -> revolute
- joint Joint4: limit lower=-3.14 upper=3.14 effort=3 velocity=120 -> lower=-3.14159 upper=3.14159 effort=3 velocity=1.5; type continuous -> revolute
- joint Joint5: limit lower=-3.14 upper=3.14 effort=3 velocity=120 -> lower=-1.5708 upper=1.5708 effort=3 velocity=1.5; type continuous -> revolute
- joint Joint6: limit lower=-3.14 upper=3.14 effort=0.8 velocity=150 -> lower=-3.14159 upper=3.14159 effort=0.8 velocity=1.8; type continuous -> revolute

Commit message: update urdf

File: robotic_arm_v4_urdf/urdf/robotic_arm_v4_urdf.urdf (robot description, URDF)
Before this commit: robot robotic_arm_v4_urdf, 7 links, 6 joints
Links:
- link End_Effector: geometry collision box size=0.12 0.14 0.06; visual mesh filename=package://robotic_arm_v4_urdf/meshes/End_Effector.STL
Joints:
- joint Joint6: axis 0 1 0 -> 1 0 0; origin xyz=0 0.0283977850233832 0 rpy=3.14159265358975 0 -3.14159265358979 -> xyz=0 0.1283977850233832 0 rpy=1.5707 0 1.5707

Commit message: updated arm speed

File: robotic_arm_v4_urdf/urdf/robotic_arm_v4_urdf.urdf (robot description, URDF)
Before this commit: robot robotic_arm_v4_urdf, 7 links, 6 joints
Joints:
- joint Joint1: limit lower=-3.14159 upper=3.14159 effort=6 velocity=1.2 -> lower=-3.14159 upper=3.14159 effort=6 velocity=3.0
- joint Joint2: limit lower=-1.5708 upper=1.5708 effort=40 velocity=1.2 -> lower=-1.5708 upper=1.5708 effort=40 velocity=3.0
- joint Joint3: limit lower=-1.20 upper=4.0 effort=40 velocity=1.2 -> lower=-1.20 upper=4.0 effort=40 velocity=3.0
- joint Joint4: limit lower=-3.14159 upper=3.14159 effort=3 velocity=1.5 -> lower=-3.14159 upper=3.14159 effort=3 velocity=4.0
- joint Joint5: limit lower=-1.5708 upper=1.5708 effort=3 velocity=1.5 -> lower=-1.5708 upper=1.5708 effort=3 velocity=4.0
- joint Joint6: limit lower=-3.14159 upper=3.14159 effort=0.8 velocity=1.8 -> lower=-3.14159 upper=3.14159 effort=0.8 velocity=5.0

Commit message: updated a new mining mechanism using space mouse

File: robotic_arm_v4_urdf/urdf/robotic_arm_v4_urdf.urdf (robot description, URDF)
Before this commit: robot robotic_arm_v4_urdf, 7 links, 6 joints
Joints:
- joint Joint5: limit lower=-1.5708 upper=1.5708 effort=3 velocity=4.0 -> lower=-2.6180 upper=2.6180 effort=3 velocity=4.0

Commit message: added loggings

File: robotic_arm_v4_urdf/urdf/robotic_arm_v4_urdf.urdf (robot description, URDF)
Before this commit: robot robotic_arm_v4_urdf, 7 links, 6 joints
Joints:
- joint Joint3: limit lower=-1.20 upper=4.0 effort=40 velocity=3.0 -> lower=-1.40 upper=4.0 effort=40 velocity=3.0
